File: USB_Backplane/Backplane.brd (EAGLE design)
At the start: 72 x 507.4 mm, 0 parts

Commit message: started electronics
Parts:
- added J10, J11, J12, J13, J14, J15, J16, J17, J18, J19, J20, J21, J22, J3, J4, J5, J6, J7, J8, J9: (no value), SparkFun-Connectors:JST-4-PTH-VERT
- added SV1, SV10, SV11, SV12, SV13, SV14, SV15, SV16, SV17, SV18, SV19, SV2, SV20, SV3, SV4, SV5, SV6, SV7, SV8, SV9: (no value), con-ml:ML40

Commit message: did some stuff
Parts:
- removed J10, J11, J12, J13, J14, J15, J16, J17, J18, J19, J20, J21, J22, J3, J4, J5, J6, J7, J8, J9: (no value), SparkFun-Connectors:JST-4-PTH-VERT
- removed SV1, SV10, SV11, SV12, SV13, SV14, SV15, SV16, SV17, SV18, SV19, SV2, SV20, SV3, SV4, SV5, SV6, SV7, SV8, SV9: (no value), con-ml:ML40
- added HUB1-1, HUB1-2, HUB1-3, HUB1-4, HUB1-5, HUB1-6, HUB1-7, HUB2-1, HUB2-2, HUB2-3, HUB2-4, HUB2-5, HUB2-6, HUB2-7, M_IN, M_OUT1, M_OUT2: (no value), SparkFun-Connectors:JST-4-PTH-VERT
- added IC1: TUSB2046BVFR, texas:VF_S-PQFP-G32
- added IC2, IC3: TUSB2077APTR, SamacSys_Parts:QFP50P900X900X160-48N
Connections:
- new net D+: M_IN.3, M_OUT1.3, M_OUT2.3
- new net D-: M_IN.2, M_OUT1.2, M_OUT2.2
- new net GND: IC1.28, IC1.7, M_IN.4, M_OUT1.4, M_OUT2.4
- new net VCC: IC1.25, IC1.3
- new net VUSB: M_IN.1, M_OUT1.1, M_OUT2.1
Other:
- board size 72 x 507.4 mm -> 72 x 371.5 mm

Commit message: Started layout
Parts:
- added IC4, IC5, IC6: LD117AS12TR, v-reg:SOT223
- added J2: 641737-1, SamacSys_Parts:641737-1
- moved M_IN 25.5 mm to (39.4, 364.5)
- moved M_OUT2 21.1 mm to (64.8, 342.9)
- moved M_OUT1 21.1 mm to (64.8, 349.2)
- moved IC1 15.3 mm to (44.5, 350.5)
- moved HUB1-1 12.7 mm to (6.35, 331.5)
Connections:
- new net 12V: J2.4
- new net 5V: IC4.3, IC5.3, IC6.3, J2.1
- new net GND1: J2.3
- new net HUB1_VCC: IC5.4
- new net HUB2_VCC: IC6.4
- new net VCC_MASTER: IC4.4
- net GND: now also IC4.1, IC5.1, IC6.1, J2.2
Routing:
- net 5V: track 0.00 -> 365.1 mm
