File: USB_Backplane/Backplane.sch (EAGLE design)
At the start: 40 parts

Commit message: did some stuff
Parts:
- removed J10, J11, J12, J13, J14, J15, J16, J17, J18, J19, J20, J21, J22, J3, J4, J5, J6, J7, J8, J9: (no value), SparkFun-Connectors:CONN_04JST-PTH-VERT
- removed SV1, SV10, SV11, SV12, SV13, SV14, SV15, SV16, SV17, SV18, SV19, SV2, SV20, SV3, SV4, SV5, SV6, SV7, SV8, SV9: (no value), con-ml:ML40
- added HUB1-1, HUB1-2, HUB1-3, HUB1-4, HUB1-5, HUB1-6, HUB1-7, HUB2-1, HUB2-2, HUB2-3, HUB2-4, HUB2-5, HUB2-6, HUB2-7, M_IN, M_OUT1, M_OUT2: (no value), SparkFun-Connectors:CONN_04JST-PTH-VERT
- added IC1: TUSB2046BVFR, texas:TUSB2046BVFR
- added IC2, IC3: TUSB2077APTR, SamacSys_Parts:TUSB2077APTR
Connections:
- new net D+: M_IN.3, M_OUT1.3, M_OUT2.3
- new net D-: M_IN.2, M_OUT1.2, M_OUT2.2
- new net GND: M_IN.4, M_OUT1.4, M_OUT2.4
- new net VUSB: M_IN.1, M_OUT1.1, M_OUT2.1
Other:
- note added: "USB IN"
- note added: "USB OUT"

Commit message: Started layout
Parts:
- added IC4, IC5, IC6: LD117AS12TR, v-reg:LD117AS12TR
- added J2: 641737-1, SamacSys_Parts:641737-1
Connections:
- new net 12V: J2.4
- new net 5V: IC4.IN, IC5.IN, IC6.IN, J2.1
- new net GND1: J2.3
- new net HUB1_VCC: IC5.OUT
- new net HUB2_VCC: IC6.OUT
- new net VCC_MASTER: IC4.OUT
- net GND: now also IC4.ADJ, IC5.ADJ, IC6.ADJ, J2.2
Changed lines of the file:
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@@
 <part name="IC2" library="SamacSys_Parts" deviceset="TUSB2077APTR" device=""/>
 <part name="IC3" library="SamacSys_Parts" deviceset="TUSB2077APTR" device=""/>
+<part name="J2" library="SamacSys_Parts" deviceset="641737-1" device=""/>
+<part name="IC4" library="v-reg" library_urn="urn:adsk.eagle:library:409" deviceset="LD117A?*" device="S" package3d_urn="urn:adsk.eagle:package:30370/1" technology="12TR"/>
+<part name="SUPPLY5" library="SparkFun-PowerSymbols" library_urn="urn:adsk.eagle:library:530" deviceset="5V" device=""/>
+<part name="GND12" library="supply1" library_urn="urn:adsk.eagle:library:371" deviceset="GND" device=""/>
+<part name="IC5" library="v-reg" library_urn="urn:adsk.eagle:library:409" deviceset="LD117A?*" device="S" package3d_urn="urn:adsk.eagle:package:30370/1" technology="12TR"/>
+<part name="SUPPLY1" library="SparkFun-PowerSymbols" library_urn="urn:adsk.eagle:library:530" deviceset="5V" device=""/>
+<part name="GND1" library="supply1" library_urn="urn:adsk.eagle:library:371" deviceset="GND" device=""/>
+<part name="IC6" library="v-reg" library_urn="urn:adsk.eagle:library:409" deviceset="LD117A?*" device="S" package3d_urn="urn:adsk.eagle:package:30370/1" technology="12TR"/>
+<part name="SUPPLY2" library="SparkFun-PowerSymbols" library_urn="urn:adsk.eagle:library:530" deviceset="5V" device=""/>
+<part name="GND2" library="supply1" library_urn="urn:adsk.eagle:library:371" deviceset="GND" device=""/>
 </parts>
 <sheets>
+<sheet>
+<description>Power Supply</description>
+<plain>
+</plain>
+<instances>
+<instance part="J2" gate="G$1" x="15.24" y="20.32" smashed="yes">
+<attribute name="NAME" x="16.51" y="25.4" size="1.778" layer="95" align="center-left"/>
+<attribute name="VALUE" x="24.13" y="25.4" size="1.778" layer="96" align="center-left"/>
+</instance>
+</instances>
+<busses>
+</busses>
+<nets>
+<net name="GND" class="0">
+<segment>
+<pinref part="J2" gate="G$1" pin="2"/>
+<wire x1="35.56" y1="20.32" x2="43.18" y2="20.32" width="0.1524" layer="91"/>
+<label x="38.1" y="20.32" size="1.778" layer="95"/>
+</segment>
+</net>
+<net name="GND1" class="0">
+<segment>
+<pinref part="J2" gate="G$1" pin="3"/>
+<wire x1="15.24" y1="17.78" x2="10.16" y2="17.78" width="0.1524" layer="91"/>
+<label x="10.16" y="17.78" size="1.778" layer="95"/>
+</segment>
+</net>
+<net name="5V" class="0">
+<segment>
+<pinref part="J2" gate="G$1" pin="1"/>
+<wire x1="15.24" y1="20.32" x2="10.16" y2="20.32" width="0.1524" layer="91"/>
+<label x="10.16" y="20.32" size="1.778" layer="95"/>
+</segment>
+</net>
+<net name="12V" class="0">
+<segment>
+<pinref part="J2" gate="G$1" pin="4"/>
+<wire x1="35.56" y1="17.78" x2="43.18" y2="17.78" width="0.1524" layer="91"/>
+<label x="38.1" y="17.78" size="1.778" layer="95"/>
+</segment>
+</net>
+</nets>
+</sheet>
 <sheet>
 <description>Master Hub</description>
@@
 <attribute name="VALUE" x="7.62" y="7.62" size="1.778" layer="96"/>
 </instance>
+<instance part="IC4" gate="G$1" x="129.54" y="71.12" smashed="yes">
+<attribute name="NAME" x="132.08" y="63.5" size="1.778" layer="95"/>
+<attribute name="VALUE" x="132.08" y="60.96" size="1.778" layer="96"/>
+</instance>
+<instance part="SUPPLY5" gate="G$1" x="119.38" y="73.66" smashed="yes">
+<attribute name="VALUE" x="119.38" y="76.454" size="1.778" layer="96" align="bottom-center"/>
+</instance>
+<instance part="GND12" gate="1" x="129.54" y="58.42" smashed="yes">
+<attribute name="VALUE" x="127" y="55.88" size="1.778" layer="96"/>
+</instance>
 </instances>
 <busses>
@@
 <label x="81.28" y="53.34" size="1.778" layer="95" rot="R180"/>
 </segment>
+<segment>
+<pinref part="GND12" gate="1" pin="GND"/>
+<pinref part="IC4" gate="G$1" pin="ADJ"/>
+<wire x1="129.54" y1="60.96" x2="129.54" y2="63.5" width="0.1524" layer="91"/>
+</segment>
 </net>
 <net name="VUSB" class="0">
@@
 <wire x1="81.28" y1="55.88" x2="68.58" y2="55.88" width="0.1524" layer="91"/>
 <label x="76.2" y="55.88" size="1.778" layer="95"/>
+</segment>
+</net>
+<net name="5V" class="0">
+<segment>
+<wire x1="119.38" y1="71.12" x2="119.38" y2="73.66" width="0.1524" layer="91"/>
+<pinref part="SUPPLY5" gate="G$1" pin="5V"/>
+<pinref part="IC4" gate="G$1" pin="IN"/>
+<wire x1="119.38" y1="71.12" x2="121.92" y2="71.12" width="0.1524" layer="91"/>
+</segment>
+</net>
+<net name="VCC_MASTER" class="0">
+<segment>
+<pinref part="IC4" gate="G$1" pin="OUT"/>
+<wire x1="137.16" y1="71.12" x2="152.4" y2="71.12" width="0.1524" layer="91"/>
+<label x="137.16" y="71.12" size="1.778" layer="95"/>
 </segment>
 </net>
@@
 <attribute name="VALUE" x="54.61" y="149.86" size="1.778" layer="96" align="center-left"/>
 </instance>
+<instance part="IC5" gate="G$1" x="-40.64" y="154.94" smashed="yes">
+<attribute name="NAME" x="-38.1" y="147.32" size="1.778" layer="95"/>
+<attribute name="VALUE" x="-38.1" y="144.78" size="1.778" layer="96"/>
+</instance>
+<instance part="SUPPLY1" gate="G$1" x="-50.8" y="157.48" smashed="yes">
+<attribute name="VALUE" x="-50.8" y="160.274" size="1.778" layer="96" align="bottom-center"/>
+</instance>
+<instance part="GND1" gate="1" x="-40.64" y="142.24" smashed="yes">
+<attribute name="VALUE" x="-43.18" y="139.7" size="1.778" layer="96"/>
+</instance>
 </instances>
 <busses>
 </busses>
 <nets>
+<net name="GND" class="0">
+<segment>
+<pinref part="GND1" gate="1" pin="GND"/>
+<pinref part="IC5" gate="G$1" pin="ADJ"/>
+<wire x1="-40.64" y1="144.78" x2="-40.64" y2="147.32" width="0.1524" layer="91"/>
+</segment>
+</net>
+<net name="5V" class="0">
+<segment>
+<wire x1="-50.8" y1="154.94" x2="-50.8" y2="157.48" width="0.1524" layer="91"/>
+<pinref part="SUPPLY1" gate="G$1" pin="5V"/>
+<pinref part="IC5" gate="G$1" pin="IN"/>
+<wire x1="-50.8" y1="154.94" x2="-48.26" y2="154.94" width="0.1524" layer="91"/>
+</segment>
+</net>
+<net name="HUB1_VCC" class="0">
+<segment>
+<pinref part="IC5" gate="G$1" pin="OUT"/>
+<wire x1="-33.02" y1="154.94" x2="-17.78" y2="154.94" width="0.1524" layer="91"/>
+<label x="-30.48" y="154.94" size="1.778" layer="95"/>
+</segment>
+</net>
 </nets>
 </sheet>
@@
 <attribute name="VALUE" x="62.23" y="101.6" size="1.778" layer="96" align="center-left"/>
 </instance>
+<instance part="IC6" gate="G$1" x="-27.94" y="93.98" smashed="yes">
+<attribute name="NAME" x="-25.4" y="86.36" size="1.778" layer="95"/>
+<attribute name="VALUE" x="-25.4" y="83.82" size="1.778" layer="96"/>
+</instance>
+<instance part="SUPPLY2" gate="G$1" x="-38.1" y="96.52" smashed="yes">
+<attribute name="VALUE" x="-38.1" y="99.314" size="1.778" layer="96" align="bottom-center"/>
+</instance>
+<instance part="GND2" gate="1" x="-27.94" y="81.28" smashed="yes">
+<attribute name="VALUE" x="-30.48" y="78.74" size="1.778" layer="96"/>
+</instance>
 </instances>
 <busses>
 </busses>
 <nets>
+<net name="GND" class="0">
+<segment>
+<pinref part="GND2" gate="1" pin="GND"/>
+<pinref part="IC6" gate="G$1" pin="ADJ"/>
+<wire x1="-27.94" y1="83.82" x2="-27.94" y2="86.36" width="0.1524" layer="91"/>
+</segment>
+</net>
+<net name="5V" class="0">
+<segment>
+<wire x1="-38.1" y1="93.98" x2="-38.1" y2="96.52" width="0.1524" layer="91"/>
+<pinref part="SUPPLY2" gate="G$1" pin="5V"/>
+<pinref part="IC6" gate="G$1" pin="IN"/>
+<wire x1="-38.1" y1="93.98" x2="-35.56" y2="93.98" width="0.1524" layer="91"/>
+</segment>
+</net>
+<net name="HUB2_VCC" class="0">
+<segment>
+<pinref part="IC6" gate="G$1" pin="OUT"/>
+<wire x1="-20.32" y1="93.98" x2="-2.54" y2="93.98" width="0.1524" layer="91"/>
+<label x="-17.78" y="93.98" size="1.778" layer="95"/>
+</segment>
+</net>
 </nets>
 </sheet>
